Commit message: feat: ros2_control urdf

File: ofa_visualization/urdf/materials.urdf.xacro (robot description, xacro)
@@ -1,30 +1,30 @@
 <?xml version="1.0"?>
-<robot xmlns:xacro="http://www.ros.org/wiki/xacro">
-    <material name="black">
-        <color rgba="0 0 0 ${255/255}" />
-    </material>
-    <material name="dark_grey">
-        <color rgba="0 0 ${155/255} ${255/255}" />
-    </material>
-    <material name="blue">
-        <color rgba="0 0 ${200/255} ${255/255}" />
-    </material>
-    <material name="green">
-        <color rgba="0 ${200/255} 0 ${255/255}" />
-    </material>
-    <material name="grey">
-        <color rgba="${50/255} ${50/255} ${50/255} ${255/255}" />
-    </material>
-    <material name="orange">
-        <color rgba="${255/255} ${108/255} ${10/255} ${255/255}" />
-    </material>
-    <material name="brown">
-        <color rgba="${222/255} ${207/255} ${195/255} ${255/255}" />
-    </material>
-    <material name="red">
-        <color rgba="${200/255} 0 0 ${255/255}" />
-    </material>
-    <material name="white">
-        <color rgba="${255/255} ${255/255} ${255/255} ${255/255}" />
-    </material>
+<robot>
+  <material name="black">
+    <color rgba="0 0 0 ${255/255}" />
+  </material>
+  <material name="dark_grey">
+    <color rgba="0 0 ${155/255} ${255/255}" />
+  </material>
+  <material name="blue">
+    <color rgba="0 0 ${200/255} ${255/255}" />
+  </material>
+  <material name="green">
+    <color rgba="0 ${200/255} 0 ${255/255}" />
+  </material>
+  <material name="grey">
+    <color rgba="${50/255} ${50/255} ${50/255} ${255/255}" />
+  </material>
+  <material name="orange">
+    <color rgba="${255/255} ${108/255} ${10/255} ${255/255}" />
+  </material>
+  <material name="brown">
+    <color rgba="${222/255} ${207/255} ${195/255} ${255/255}" />
+  </material>
+  <material name="red">
+    <color rgba="${200/255} 0 0 ${255/255}" />
+  </material>
+  <material name="white">
+    <color rgba="${255/255} ${255/255} ${255/255} ${255/255}" />
+  </material>
 </robot>
