Commit message: feat: nonblocking read

File: ofa_description/ros2_control/2dof_arm.ros2_control.xacro (robot description, xacro)
@@ -6,5 +6,5 @@
         <hardware>
           <plugin>cubemars_hardware/CubeMarsSystemHardware</plugin>
-          <param name="can">can0</param>
+          <param name="can_interface">can0</param>
         </hardware>
       </xacro:unless>
@@ -16,13 +16,22 @@
       </xacro:if>
       <joint name="${prefix}joint2">
-        <param name="can_id">0</param>
+        <param name="can_id">90</param>
+        <param name="pole_pairs">21</param>
+        <param name="reduction_ratio">9</param>
+        <param name="kt">0.123</param>
         <command_interface name="position" />
         <state_interface name="position" />
+        <state_interface name="velocity" />
+        <state_interface name="effort" />
       </joint>
-      <joint name="${prefix}joint3">
-        <param name="can_id">1</param>
+      <!-- <joint name="${prefix}joint3">
+        <param name="can_id">91</param>
+        <param name="pole_pairs">21</param>
+        <param name="reduction_ratio">9</param>
+        <param name="kt">0.123</param>
         <command_interface name="position" />
         <state_interface name="position" />
-      </joint>
+        <state_interface name="velocity" />
+      </joint> -->
     </ros2_control>
   </xacro:macro>

Commit message: fix: read

File: ofa_description/ros2_control/2dof_arm.ros2_control.xacro (robot description, xacro)
@@ -25,5 +25,5 @@
         <state_interface name="effort" />
       </joint>
-      <!-- <joint name="${prefix}joint3">
+      <joint name="${prefix}joint3">
         <param name="can_id">91</param>
         <param name="pole_pairs">21</param>
@@ -33,5 +33,5 @@
         <state_interface name="position" />
         <state_interface name="velocity" />
-      </joint> -->
+      </joint>
     </ros2_control>
   </xacro:macro>

Commit message: feat: command mode switch

File: ofa_description/ros2_control/2dof_arm.ros2_control.xacro (robot description, xacro)
@@ -1,18 +1,10 @@
 <?xml version="1.0"?>
 <robot xmlns:xacro="http://www.ros.org/wiki/xacro">
-  <xacro:macro name="arm_ros2_control" params="name prefix use_mock_hardware">
+  <xacro:macro name="arm_ros2_control" params="name prefix">
     <ros2_control name="${name}" type="system">
-      <xacro:unless value="${use_mock_hardware}">
-        <hardware>
-          <plugin>cubemars_hardware/CubeMarsSystemHardware</plugin>
-          <param name="can_interface">can0</param>
-        </hardware>
-      </xacro:unless>
-      <xacro:if value="${use_mock_hardware}">
-        <hardware>
-          <plugin>mock_components/GenericSystem</plugin>
-          <param name="calculate_dynamics">true</param>
-        </hardware>
-      </xacro:if>
+      <hardware>
+        <plugin>cubemars_hardware/CubeMarsSystemHardware</plugin>
+        <param name="can_interface">can0</param>
+      </hardware>
       <joint name="${prefix}joint2">
         <param name="can_id">90</param>
@@ -20,8 +12,4 @@
         <param name="reduction_ratio">10</param>
         <param name="kt">0.123</param>
-        <command_interface name="position" />
-        <state_interface name="position" />
-        <state_interface name="velocity" />
-        <state_interface name="effort" />
       </joint>
       <joint name="${prefix}joint3">
@@ -30,7 +18,4 @@
         <param name="reduction_ratio">10</param>
         <param name="kt">0.123</param>
-        <command_interface name="position" />
-        <state_interface name="position" />
-        <state_interface name="velocity" />
       </joint>
     </ros2_control>

File: ofa_description/urdf/robot.urdf.xacro (robot description, xacro)
@@ -4,5 +4,4 @@
   <!-- Enable setting arguments from the launch file -->
   <xacro:arg name="prefix" default="" />
-  <xacro:arg name="use_mock_hardware" default="false" />
   <!-- Import robot macro -->
    <xacro:include filename="robot_description.urdf.xacro" />
@@ -17,5 +16,5 @@
   <xacro:weed_robot parent="world" prefix="$(arg prefix)" />
   <xacro:arm_ros2_control
-    name="2dof_arm" prefix="$(arg prefix)" use_mock_hardware="$(arg use_mock_hardware)"/>
+    name="2dof_arm" prefix="$(arg prefix)" />
   <!-- <xacro:linear_axis_ros2_control name="linear_axis" prefix="$(arg prefix)" /> -->
 </robot>

File: ofa_description/urdf/robot_description.urdf.xacro (robot description, xacro)
@@ -68,5 +68,5 @@
 		<child link="${prefix}link2" />
 		<axis xyz="1 0 0" />
-		<limit lower="${-pi/2}" upper="${pi/2}" velocity="100" effort="100" />
+		<limit lower="${-pi}" upper="${pi}" velocity="5" effort="10" />
 	</joint>
 	<xacro:property name="arm_length" value="0.25" />
@@ -101,4 +101,5 @@
 		<child link="${prefix}link3" />
 		<axis xyz="1 0 0" />
+		<limit lower="${-pi}" upper="${pi}" velocity="5" effort="10" />
 	</joint>
 	<link name="${prefix}link3">

Commit message: feat: mock hardware

File: ofa_description/ros2_control/2dof_arm.ros2_control.xacro (robot description, xacro)
@@ -1,9 +1,15 @@
 <?xml version="1.0"?>
 <robot xmlns:xacro="http://www.ros.org/wiki/xacro">
-  <xacro:macro name="arm_ros2_control" params="name prefix">
+  <xacro:macro name="arm_ros2_control" params="name prefix use_mock_hardware">
     <ros2_control name="${name}" type="system">
       <hardware>
-        <plugin>cubemars_hardware/CubeMarsSystemHardware</plugin>
-        <param name="can_interface">can0</param>
+        <xacro:if value="${use_mock_hardware}">
+          <plugin>mock_components/GenericSystem</plugin>
+          <param name="calculate_dynamics">true</param>
+        </xacro:if>
+        <xacro:unless value="${use_mock_hardware}">
+          <plugin>cubemars_hardware/CubeMarsSystemHardware</plugin>
+          <param name="can_interface">can0</param>
+        </xacro:unless>
       </hardware>
       <joint name="${prefix}joint2">
@@ -12,4 +18,12 @@
         <param name="gear_ratio">10</param>
         <param name="kt">0.123</param>
+        <command_interface name="position"/>
+        <command_interface name="velocity"/>
+        <command_interface name="acceleration"/>
+        <command_interface name="effort"/>
+        <state_interface name="position"/>
+        <state_interface name="velocity"/>
+        <state_interface name="effort"/>
+        <state_interface name="temperature"/>
       </joint>
       <joint name="${prefix}joint3">
@@ -18,4 +32,12 @@
         <param name="gear_ratio">10</param>
         <param name="kt">0.123</param>
+        <command_interface name="position"/>
+        <command_interface name="velocity"/>
+        <command_interface name="acceleration"/>
+        <command_interface name="effort"/>
+        <state_interface name="position"/>
+        <state_interface name="velocity"/>
+        <state_interface name="effort"/>
+        <state_interface name="temperature"/>
       </joint>
     </ros2_control>

File: ofa_description/urdf/robot.urdf.xacro (robot description, xacro)
@@ -4,4 +4,5 @@
   <!-- Enable setting arguments from the launch file -->
   <xacro:arg name="prefix" default="" />
+  <xacro:arg name="use_mock_hardware" default="false" />
   <!-- Import robot macro -->
    <xacro:include filename="robot_description.urdf.xacro" />
@@ -16,5 +17,5 @@
   <xacro:weed_robot parent="world" prefix="$(arg prefix)" />
   <xacro:arm_ros2_control
-    name="2dof_arm" prefix="$(arg prefix)" />
+    name="2dof_arm" prefix="$(arg prefix)" use_mock_hardware="$(arg use_mock_hardware)"/>
   <!-- <xacro:linear_axis_ros2_control name="linear_axis" prefix="$(arg prefix)" /> -->
 </robot>
