Commit message: feat: teknic_hardware init

File: ofa_description/ros2_control/arm_2dof.ros2_control.xacro (robot description, xacro)
@@ -1,10 +1,9 @@
 <?xml version="1.0"?>
 <robot xmlns:xacro="http://www.ros.org/wiki/xacro">
-  <xacro:macro name="arm_ros2_control" params="name prefix use_mock_hardware">
+  <xacro:macro name="arm_2dof_ros2_control" params="name prefix use_mock_hardware">
     <ros2_control name="${name}" type="system">
       <hardware>
         <xacro:if value="${use_mock_hardware}">
           <plugin>mock_components/GenericSystem</plugin>
-          <param name="calculate_dynamics">true</param>
         </xacro:if>
         <xacro:unless value="${use_mock_hardware}">

File: ofa_description/urdf/robot.urdf.xacro (robot description, xacro)
@@ -11,11 +11,12 @@
   <xacro:include filename="materials.urdf.xacro" />
   <!-- Import ros2_control description -->
-  <xacro:include filename="$(find ofa_description)/ros2_control/2dof_arm.ros2_control.xacro" />
-  <!-- <xacro:include filename="$(find ofa_description)/ros2_control/linear_axis.ros2_control.xacro" /> -->
+  <xacro:include filename="$(find ofa_description)/ros2_control/arm_2dof.ros2_control.xacro" />
+  <xacro:include filename="$(find ofa_description)/ros2_control/linear_axis.ros2_control.xacro" />
   <!-- Used for fixing robot -->
   <link name="world"/>
   <xacro:weed_robot parent="world" prefix="$(arg prefix)" />
-  <xacro:arm_ros2_control
-    name="2dof_arm" prefix="$(arg prefix)" use_mock_hardware="$(arg use_mock_hardware)"/>
-  <!-- <xacro:linear_axis_ros2_control name="linear_axis" prefix="$(arg prefix)" /> -->
+  <xacro:arm_2dof_ros2_control
+    name="arm_2dof" prefix="$(arg prefix)" use_mock_hardware="$(arg use_mock_hardware)"/>
+  <xacro:linear_axis_ros2_control
+    name="linear_axis" prefix="$(arg prefix)" use_mock_hardware="$(arg use_mock_hardware)"/>
 </robot>

Commit message: fix: moveit demo

File: ofa_description/ros2_control/arm_2dof.ros2_control.xacro (robot description, xacro)
@@ -1,5 +1,5 @@
 <?xml version="1.0"?>
 <robot xmlns:xacro="http://www.ros.org/wiki/xacro">
-  <xacro:macro name="arm_2dof_ros2_control" params="name prefix use_mock_hardware">
+  <xacro:macro name="arm_2dof_ros2_control" params="name use_mock_hardware">
     <ros2_control name="${name}" type="system">
       <hardware>
@@ -12,5 +12,5 @@
         </xacro:unless>
       </hardware>
-      <joint name="${prefix}joint2">
+      <joint name="joint2">
         <param name="can_id">90</param>
         <param name="pole_pairs">21</param>
@@ -26,5 +26,5 @@
         <state_interface name="temperature"/>
       </joint>
-      <joint name="${prefix}joint3">
+      <joint name="joint3">
         <param name="can_id">91</param>
         <param name="pole_pairs">21</param>

File: ofa_description/ros2_control/linear_axis.ros2_control.xacro (robot description, xacro)
@@ -1,15 +1,15 @@
 <?xml version="1.0"?>
 <robot xmlns:xacro="http://www.ros.org/wiki/xacro">
-  <xacro:macro name="linear_axis_ros2_control" params="name prefix use_mock_hardware">
+  <xacro:macro name="linear_axis_ros2_control" params="name use_mock_hardware">
     <ros2_control name="${name}" type="system">
       <hardware>
-        <xacro:if value="${use_mock_hardware}">
+        <!-- <xacro:if value="${use_mock_hardware}"> -->
           <plugin>mock_components/GenericSystem</plugin>
-        </xacro:if>
+        <!-- </xacro:if>
         <xacro:unless value="${use_mock_hardware}">
           <plugin>teknic_hardware/TeknicSystemHardware</plugin>
-        </xacro:unless>
+        </xacro:unless> -->
       </hardware>
-      <joint name="${prefix}joint1">
+      <joint name="joint1">
         <command_interface name="position"/>
         <command_interface name="velocity"/>

File: ofa_description/urdf/inertia.urdf.xacro (robot description, xacro)
@@ -1,33 +1,33 @@
 <?xml version="1.0"?>
 <robot xmlns:xacro="http://www.ros.org/wiki/xacro">
-    <xacro:macro name="cylinder_inertia" params="m r h">
-        <inertia
-            ixx="${m*(3*r*r+h*h)/12}"
-            ixy="0"
-            ixz="0"
-            iyy="${m*(3*r*r+h*h)/12}"
-            iyz="0"
-            izz="${m*r*r/2}"
-        />
-    </xacro:macro>
-    <xacro:macro name="box_inertia" params="m x y z">
-        <inertia
-            ixx="${m*(y*y+z*z)/12}"
-            ixy="0"
-            ixz="0"
-            iyy="${m*(x*x+z*z)/12}"
-            iyz="0"
-            izz="${m*(x*x+z*z)/12}"
-        />
-    </xacro:macro>
-    <xacro:macro name="sphere_inertia" params="m r">
-        <inertia
-            ixx="${2*m*r*r/5}"
-            ixy="0"
-            ixz="0"
-            iyy="${2*m*r*r/5}"
-            iyz="0"
-            izz="${2*m*r*r/5}"
-        />
-    </xacro:macro>
+  <xacro:macro name="cylinder_inertia" params="m r h">
+    <inertia
+      ixx="${m*(3*r*r+h*h)/12}"
+      ixy="0"
+      ixz="0"
+      iyy="${m*(3*r*r+h*h)/12}"
+      iyz="0"
+      izz="${m*r*r/2}"
+    />
+  </xacro:macro>
+  <xacro:macro name="box_inertia" params="m x y z">
+    <inertia
+      ixx="${m*(y*y+z*z)/12}"
+      ixy="0"
+      ixz="0"
+      iyy="${m*(x*x+z*z)/12}"
+      iyz="0"
+      izz="${m*(x*x+y*y)/12}"
+    />
+  </xacro:macro>
+  <xacro:macro name="sphere_inertia" params="m r">
+    <inertia
+      ixx="${2*m*r*r/5}"
+      ixy="0"
+      ixz="0"
+      iyy="${2*m*r*r/5}"
+      iyz="0"
+      izz="${2*m*r*r/5}"
+    />
+  </xacro:macro>
 </robot>

File: ofa_description/urdf/robot.urdf.xacro (robot description, xacro)
@@ -1,7 +1,6 @@
 <?xml version="1.0"?>
 <!-- Weed Control Unit Robot Arm -->
-<robot xmlns:xacro="http://www.ros.org/wiki/xacro" name="weed_arm">
+<robot xmlns:xacro="http://www.ros.org/wiki/xacro" name="ofa_arm">
   <!-- Enable setting arguments from the launch file -->
-  <xacro:arg name="prefix" default="" />
   <xacro:arg name="use_mock_hardware" default="false" />
   <!-- Import robot macro -->
@@ -15,8 +14,8 @@
   <!-- Used for fixing robot -->
   <link name="world"/>
-  <xacro:weed_robot parent="world" prefix="$(arg prefix)" />
+  <xacro:weed_robot parent="world" />
   <xacro:arm_2dof_ros2_control
-    name="arm_2dof" prefix="$(arg prefix)" use_mock_hardware="$(arg use_mock_hardware)"/>
+    name="arm_2dof" use_mock_hardware="$(arg use_mock_hardware)"/>
   <xacro:linear_axis_ros2_control
-    name="linear_axis" prefix="$(arg prefix)" use_mock_hardware="$(arg use_mock_hardware)"/>
+    name="linear_axis" use_mock_hardware="$(arg use_mock_hardware)"/>
 </robot>

File: ofa_description/urdf/robot_description.urdf.xacro (robot description, xacro)
@@ -1,18 +1,18 @@
 <?xml version="1.0"?>
 <robot xmlns:xacro="http://www.ros.org/wiki/xacro">
-  <xacro:macro name="weed_robot" params="parent prefix">
+  <xacro:macro name="weed_robot" params="parent">
 	<xacro:property name="attachment_off" value="${0.06+0.002}" />
 	<xacro:property name="tube_off" value="${0.01}" />
 	<xacro:property name="height" value="${0.5+attachment_off}" />
-	<joint name="${prefix}base_joint" type="fixed">
+	<joint name="base_joint" type="fixed">
 		<origin xyz="0 0 ${height}" rpy="0 0 0" />
 		<parent link="${parent}" />
-		<child link="${prefix}base_link" />
+		<child link="base_link" />
 	</joint>
 	<xacro:property name="base_l" value="1.216" />
 	<xacro:property name="base_w" value="0.06" />
 	<xacro:property name="base_h" value="0.072" />
-	<xacro:property name="base_m" value="5" />
-	<link name="${prefix}base_link">
+	<xacro:property name="base_m" value="6" />
+	<link name="base_link">
 		<visual>
 			<origin xyz="0 0 ${base_h/2}" rpy="0 0 0" />
@@ -35,15 +35,15 @@
 	</link>
 	<xacro:property name="axis_length" value="1" />
-	<joint name="${prefix}joint1" type="prismatic">
+	<joint name="joint1" type="prismatic">
 		<origin xyz="${-base_l/2+0.116} 0 ${-attachment_off}" rpy="0 0 0" />
-		<parent link="${prefix}base_link" />
-		<child link="${prefix}link1" />
+		<parent link="base_link" />
+		<child link="link1" />
 		<axis xyz="1 0 0" />
-		<limit lower="0" upper="${axis_length}" velocity="1" effort="10" />
+		<limit lower="0" upper="${axis_length}" velocity="1.0" effort="10" />
 	</joint>
 	<xacro:property name="motor_r" value="${0.089/2}" />
 	<xacro:property name="motor_h" value="0.05025" />
 	<xacro:property name="motor_m" value="0.521" />
-	<link name="${prefix}link1">
+	<link name="link1">
 		<visual>
 			<origin xyz="0 0 0" rpy="0 ${pi/2} 0" />
@@ -65,15 +65,15 @@
 		</inertial>
 	</link>
-	<xacro:property name="camera_w" value="0.120" />
-	<xacro:property name="camera_h" value="0.080" />
+	<xacro:property name="camera_w" value="0.12" />
+	<xacro:property name="camera_h" value="0.08" />
 	<xacro:property name="camera_l" value="0.048" />
 	<xacro:property name="camera_m" value="0.335" />
 	<xacro:property name="camera_off" value="${0.0885/2+0.002}" />
-	<joint name="${prefix}joint1_camera" type="fixed">
+	<joint name="joint1_camera" type="fixed">
 		<origin xyz="-${camera_off} 0 ${attachment_off}" rpy="0 0 0" />
-		<parent link="${prefix}link1" />
-		<child link="${prefix}link1_camera" />
-	</joint>
-	<link name="${prefix}link1_camera">
+		<parent link="link1" />
+		<child link="link1_camera" />
+	</joint>
+	<link name="link1_camera">
 		<visual>
 			<origin xyz="${-camera_l/2} 0 ${-camera_h/2}" rpy="0 0 0" />
@@ -95,10 +95,10 @@
 		</inertial>
 	</link>
-	<joint name="${prefix}joint2" type="revolute">
+	<joint name="joint2" type="revolute">
 		<origin xyz="${motor_h/2+tube_off} 0 0" rpy="0 0 0" />
-		<parent link="${prefix}link1" />
-		<child link="${prefix}link2" />
+		<parent link="link1" />
+		<child link="link2" />
 		<axis xyz="1 0 0" />
-		<limit lower="${-pi}" upper="${pi}" velocity="5" effort="10" />
+		<limit lower="${-pi*2/3}" upper="${pi*2/3}" velocity="5.0" effort="10" />
 	</joint>
 	<xacro:property name="arm_r" value="${0.045/2}" />
@@ -108,5 +108,5 @@
 	<xacro:property name="arm2_l" value="0.425" />
 	<xacro:property name="arm2_m" value="${1650*(arm_r**2*pi-arm_ri**2*pi)*arm2_l}" />
-	<link name="${prefix}link2">
+	<link name="link2">
 		<visual>
 			<origin xyz="${arm_r} 0 ${-arm1_l/2}" rpy="0 0 0" />
@@ -128,10 +128,10 @@
 		</inertial>
 	</link>
-	<joint name="${prefix}joint2_motor" type="fixed">
+	<joint name="joint2_motor" type="fixed">
 		<origin xyz="${-motor_h/2-0.0058} 0 ${-arm1_l}" rpy="0 0 0" />
-		<parent link="${prefix}link2" />
-		<child link="${prefix}link2_motor" />
-	</joint>
-	<link name="${prefix}link2_motor">
+		<parent link="link2" />
+		<child link="link2_motor" />
+	</joint>
+	<link name="link2_motor">
 		<visual>
 			<origin xyz="0 0 0" rpy="0 ${pi/2} 0" />
@@ -153,12 +153,12 @@
 		</inertial>
 	</link>
-	<joint name="${prefix}joint3" type="continuous">
+	<joint name="joint3" type="revolute">
 		<origin xyz="${-motor_h/2-tube_off} 0 0" rpy="0 0 0" />
-		<parent link="${prefix}link2_motor" />
-		<child link="${prefix}link3" />
+		<parent link="link2_motor" />
+		<child link="link3" />
 		<axis xyz="1 0 0" />
-		<limit lower="${-pi}" upper="${pi}" velocity="5" effort="10" />
-	</joint>
-	<link name="${prefix}link3">
+		<limit lower="${-pi*2/3}" upper="${pi*2/3}" velocity="5.0" effort="10" />
+	</joint>
+	<link name="link3">
 		<visual>
 			<origin xyz="${-arm_r} 0 ${-arm2_l/2}" rpy="0 0 0" />
@@ -180,15 +180,15 @@
 		</inertial>
 	</link>
-	<joint name="${prefix}joint3_end" type="fixed">
+	<joint name="joint3_end" type="fixed">
 		<origin xyz="${-arm_r} 0 ${-arm2_l}" rpy="0 0 0" />
-		<parent link="${prefix}link3" />
-		<child link="${prefix}link3_end" />
+		<parent link="link3" />
+		<child link="link3_end" />
 	</joint>
 	<xacro:property name="end_r" value="0.005" />
-	<xacro:property name="end_l" value="0.01" />
+	<xacro:property name="end_l" value="0.02" />
 	<xacro:property name="end_m" value="1" />
-	<link name="${prefix}link3_end">
-		<visual>
-			<origin xyz="0 0 ${-end_l}" rpy="0 0 0" />
+	<link name="link3_end">
+		<visual>
+			<origin xyz="0 0 ${-end_l/2}" rpy="0 0 0" />
 			<geometry>
 				<cylinder length="${end_l}" radius="${end_r}" />
@@ -197,5 +197,5 @@
 		</visual>
 		<collision>
-			<origin xyz="0 0 ${-end_l}" rpy="0 0 0" />
+			<origin xyz="0 0 ${-end_l/2}" rpy="0 0 0" />
 			<geometry>
 				<cylinder length="${end_l}" radius="${end_r}" />
@@ -203,5 +203,5 @@
 		</collision>
 		<inertial>
-			<origin xyz="0 0 ${-end_l}" rpy="0 0 0" />
+			<origin xyz="0 0 ${-end_l/2}" rpy="0 0 0" />
 			<mass value="${end_m}" />
 			<xacro:cylinder_inertia m="${end_m}" r="${end_r}" h="${end_l}" />
@@ -216,10 +216,10 @@
 	<xacro:property name="top_h" value="${height-2*wheel_r}" />
 	<xacro:macro name="wheel" params="prefix x y">
-		<joint name="${prefix}_wheel_joint" type="fixed">
+		<joint name="_wheel_joint" type="fixed">
 			<parent link="base_link" />
-			<child link="${prefix}_wheel_link" />
+			<child link="_wheel_link" />
 			<origin xyz="${x} ${y} 0" rpy="0 0 0" />
 		</joint>
-		<link name="${prefix}_wheel_link">
+		<link name="_wheel_link">
 			<visual>
 				<origin xyz="0 0 ${-top_h/2}" rpy="0 0 0"/>

Commit message: fix: weed control

File: ofa_description/ros2_control/arm_2dof.ros2_control.xacro (robot description, xacro)
@@ -4,11 +4,11 @@
     <ros2_control name="${name}" type="system">
       <hardware>
-        <!-- <xacro:if value="${use_mock_hardware}"> -->
+        <xacro:if value="${use_mock_hardware}">
           <plugin>mock_components/GenericSystem</plugin>
-        <!-- </xacro:if>
+        </xacro:if>
         <xacro:unless value="${use_mock_hardware}">
           <plugin>cubemars_hardware/CubeMarsSystemHardware</plugin>
           <param name="can_interface">can0</param>
-        </xacro:unless> -->
+        </xacro:unless>
       </hardware>
       <joint name="joint2">

File: ofa_description/ros2_control/linear_axis.ros2_control.xacro (robot description, xacro)
@@ -4,10 +4,10 @@
     <ros2_control name="${name}" type="system">
       <hardware>
-        <!-- <xacro:if value="${use_mock_hardware}">
+        <xacro:if value="${use_mock_hardware}">
           <plugin>mock_components/GenericSystem</plugin>
         </xacro:if>
-        <xacro:unless value="${use_mock_hardware}"> -->
+        <xacro:unless value="${use_mock_hardware}">
           <plugin>teknic_hardware/TeknicSystemHardware</plugin>
-        <!-- </xacro:unless> -->
+        </xacro:unless>
       </hardware>
       <joint name="joint1">

File: ofa_description/urdf/ofa_robot_description.urdf.xacro (robot description, xacro)
@@ -156,5 +156,5 @@
     </link>
     <joint name="joint3" type="revolute">
-      <origin xyz="${-motor_h/2-tube_off} 0 0" rpy="0 0 0" />
+      <origin xyz="${-motor_h/2-tube_off} 0 0" rpy="${pi} 0 0" />
       <parent link="link2_motor" />
       <child link="link3" />

Commit message: feat: read_only

File: ofa_description/ros2_control/arm_2dof.ros2_control.xacro (robot description, xacro)
@@ -1,5 +1,5 @@
 <?xml version="1.0"?>
 <robot xmlns:xacro="http://www.ros.org/wiki/xacro">
-  <xacro:macro name="arm_2dof_ros2_control" params="name use_mock_hardware">
+  <xacro:macro name="arm_2dof_ros2_control" params="name use_mock_hardware read_only">
     <ros2_control name="${name}" type="system">
       <hardware>
@@ -18,4 +18,7 @@
         <param name="kt">0.123</param>
         <param name="enc_off">-0.084</param>
+        <xacro:if value="${read_only}">
+          <param name="read_only">1</param>
+        </xacro:if>
         <command_interface name="position"/>
         <command_interface name="velocity"/>
@@ -33,4 +36,7 @@
         <param name="kt">0.123</param>
         <param name="enc_off">-0.084</param>
+        <xacro:if value="${read_only}">
+          <param name="read_only">1</param>
+        </xacro:if>
         <command_interface name="position"/>
         <command_interface name="velocity"/>

File: ofa_description/ros2_control/linear_axis.ros2_control.xacro (robot description, xacro)
@@ -1,5 +1,5 @@
 <?xml version="1.0"?>
 <robot xmlns:xacro="http://www.ros.org/wiki/xacro">
-  <xacro:macro name="linear_axis_ros2_control" params="name use_mock_hardware">
+  <xacro:macro name="linear_axis_ros2_control" params="name use_mock_hardware read_only">
     <ros2_control name="${name}" type="system">
       <hardware>
@@ -19,4 +19,7 @@
         <param name="peak_torque">4.01</param>
         <param name="homing">1</param>
+        <xacro:if value="${read_only}">
+          <param name="read_only">1</param>
+        </xacro:if>
         <command_interface name="position"/>
         <command_interface name="velocity"/>

File: ofa_description/urdf/ofa_robot.urdf.xacro (robot description, xacro)
@@ -2,6 +2,7 @@
 <!-- Weed Control Unit Robot Arm -->
 <robot xmlns:xacro="http://www.ros.org/wiki/xacro" name="ofa_robot">
-  <!-- Enable setting arguments from the launch file -->
+  <!-- Arguments -->
   <xacro:arg name="use_mock_hardware" default="false" />
+  <xacro:arg name="read_only" default="false" />
   <!-- Import robot macro -->
    <xacro:include filename="ofa_robot_description.urdf.xacro" />
@@ -19,6 +20,6 @@
   <xacro:weed_robot parent="world" />
   <xacro:arm_2dof_ros2_control
-    name="arm_2dof" use_mock_hardware="$(arg use_mock_hardware)"/>
+    name="arm_2dof" use_mock_hardware="$(arg use_mock_hardware)" read_only="$(arg read_only)" />
   <xacro:linear_axis_ros2_control
-    name="linear_axis" use_mock_hardware="$(arg use_mock_hardware)"/>
+    name="linear_axis" use_mock_hardware="$(arg use_mock_hardware)" read_only="$(arg read_only)" />
 </robot>

File: ofa_description/urdf/ofa_robot_description.urdf.xacro (robot description, xacro)
@@ -40,5 +40,5 @@
     <xacro:property name="end_m" value="1" />
     <joint name="base_joint" type="fixed">
-      <origin xyz="0 0 ${height}" rpy="0 0 0" />
+      <origin xyz="0 0 ${height}" rpy="0 0 ${pi}" />
       <parent link="${parent}" />
       <child link="base_link" />

Commit message: feat: arm positioning

File: ofa_description/ros2_control/arm_2dof.ros2_control.xacro (robot description, xacro)
@@ -18,4 +18,5 @@
         <param name="kt">0.123</param>
         <param name="enc_off">-0.084</param>
+        <param name="trq_limit">10</param>
         <xacro:if value="${read_only}">
           <param name="read_only">1</param>
@@ -36,4 +37,5 @@
         <param name="kt">0.123</param>
         <param name="enc_off">-0.084</param>
+        <param name="trq_limit">10</param>
         <xacro:if value="${read_only}">
           <param name="read_only">1</param>

File: ofa_description/urdf/ofa_robot_description.urdf.xacro (robot description, xacro)
@@ -32,5 +32,5 @@
     <xacro:property name="motor_h" value="0.05025" />
     <!-- Offset between center of motor and center of carriage in x-direction -->
-    <xacro:property name="motor_off" value="${0.0026}" />
+    <xacro:property name="motor_off" value="${-0.0026}" />
     <!-- Camera enclosure dimensions -->
     <xacro:property name="camera_shield_w" value="0.12" />
@@ -39,6 +39,6 @@
     <xacro:property name="camera_shield_wall" value="0.002" />
     <!-- Offset between camera enclosure and motor center -->
-    <xacro:property name="camera_shield_off_x" value="${motor_h/2+0.04355}" />
-    <xacro:property name="camera_shield_off_y" value="${0.044}" />
+    <xacro:property name="camera_shield_off_x" value="${-motor_h/2-0.04355}" />
+    <xacro:property name="camera_shield_off_y" value="-0.044" />
     <!-- Camera dimensions -->
     <xacro:property name="camera_w" value="0.11526" />
@@ -52,5 +52,5 @@
     <!-- Tube dimensions -->
     <xacro:property name="arm_r" value="${0.045/2}" />
-    <xacro:property name="arm1_l" value="0.362" />
+    <xacro:property name="arm1_l" value="${0.451-2*motor_r}" />
     <xacro:property name="arm2_l" value="0.161" />
     <!-- End effector dimensions -->
@@ -107,5 +107,5 @@
     </link>
     <joint name="joint1" type="prismatic">
-      <origin xyz="${-axis_l/2+carriage_off-motor_off} 0 ${-axis_h-attachment_off}" rpy="0 0 0" />
+      <origin xyz="${-axis_l/2+carriage_off+motor_off} 0 ${-axis_h-attachment_off}" rpy="0 0 0" />
       <parent link="base_link" />
       <child link="link1" />
@@ -130,5 +130,5 @@
     </link>
     <joint name="camera_shield_joint" type="fixed">
-      <origin xyz="${-camera_shield_off_x-camera_shield_l/2} ${-camera_shield_off_y} ${attachment_off}" rpy="0 0 0" />
+      <origin xyz="${camera_shield_off_x-camera_shield_l/2} ${camera_shield_off_y} ${attachment_off}" rpy="0 0 0" />
       <parent link="link1" />
       <child link="camera_shield_link" />
@@ -163,5 +163,5 @@
     </link>
     <joint name="camera_joint" type="fixed">
-      <origin xyz="0 ${-camera_off_y} ${-camera_off_z}" rpy="0 0 0" />
+      <origin xyz="0 ${camera_off_y} ${-camera_off_z}" rpy="0 0 0" />
       <parent link="camera_shield_link" />
       <child link="camera_link" />
