Commit message: feat: add auto_create_ikfast script

File: ofa_description/urdf/ofa_robot_description.urdf.xacro (robot description, xacro)
@@ -187,10 +187,10 @@
 		<origin xyz="${-arm_r} 0 ${-arm2_l}" rpy="0 0 0" />
 		<parent link="link3" />
-		<child link="link3_end" />
+		<child link="eef_link" />
 	</joint>
 	<xacro:property name="end_r" value="0.005" />
 	<xacro:property name="end_l" value="0.02" />
 	<xacro:property name="end_m" value="1" />
-	<link name="link3_end">
+	<link name="eef_link">
 		<visual>
 			<origin xyz="0 0 ${-end_l/2}" rpy="0 0 0" />

Commit message: chore: update urdf

File: ofa_description/urdf/ofa_robot_description.urdf.xacro (robot description, xacro)
@@ -107,7 +107,7 @@
 	<xacro:property name="arm_r" value="${0.045/2}" />
 	<xacro:property name="arm_ri" value="${0.041/2}" />
-	<xacro:property name="arm1_l" value="0.25" />
+	<xacro:property name="arm1_l" value="0.368" />
 	<xacro:property name="arm1_m" value="${1650*(arm_r**2*pi-arm_ri**2*pi)*arm1_l}" />
-	<xacro:property name="arm2_l" value="0.425" />
+	<xacro:property name="arm2_l" value="0.307" />
 	<xacro:property name="arm2_m" value="${1650*(arm_r**2*pi-arm_ri**2*pi)*arm2_l}" />
 	<link name="link2">

Commit message: feat: update description

File: ofa_description/urdf/ofa_robot_description.urdf.xacro (robot description, xacro)
@@ -36,5 +36,5 @@
     <xacro:property name="axis_length" value="1" />
     <joint name="joint1" type="prismatic">
-      <origin xyz="${-base_l/2+0.116} 0 ${-attachment_off}" rpy="0 0 0" />
+      <origin xyz="${base_l/2-0.116} 0 ${-attachment_off}" rpy="0 0 0" />
       <parent link="base_link" />
       <child link="link1" />
@@ -70,7 +70,7 @@
     <xacro:property name="camera_l" value="0.048" />
     <xacro:property name="camera_m" value="0.335" />
-    <xacro:property name="camera_off" value="${0.0885/2+0.002}" />
+    <xacro:property name="camera_off" value="${0.0885/2+0.004}" />
     <joint name="joint1_camera" type="fixed">
-      <origin xyz="-${camera_off} 0 ${attachment_off}" rpy="0 0 0" />
+      <origin xyz="${camera_off} 0 ${attachment_off}" rpy="0 0 0" />
       <parent link="link1" />
       <child link="link1_camera" />
@@ -78,5 +78,5 @@
     <link name="link1_camera">
       <visual>
-        <origin xyz="${-camera_l/2} 0 ${-camera_h/2}" rpy="0 0 0" />
+        <origin xyz="${camera_l/2} 0 ${-camera_h/2}" rpy="0 0 0" />
         <geometry>
           <box size="${camera_l} ${camera_w} ${camera_h}" />
@@ -85,5 +85,5 @@
       </visual>
       <collision>
-        <origin xyz="${-camera_l/2} 0 ${-camera_h/2}" rpy="0 0 0" />
+        <origin xyz="${camera_l/2} 0 ${-camera_h/2}" rpy="0 0 0" />
         <geometry>
           <box size="${camera_l} ${camera_w} ${camera_h}" />
@@ -91,5 +91,5 @@
       </collision>
       <inertial>
-        <origin xyz="${-camera_l/2} 0 ${-camera_h/2}" rpy="0 0 0" />
+        <origin xyz="${camera_l/2} 0 ${-camera_h/2}" rpy="0 0 0" />
         <mass value="${camera_m}" />
         <xacro:box_inertia m="${camera_m}" x="${camera_l}" y="${camera_w}" z="${camera_h}" />
@@ -97,8 +97,8 @@
     </link>
     <joint name="joint2" type="revolute">
-      <origin xyz="${motor_h/2+tube_off} 0 0" rpy="0 0 0" />
+      <origin xyz="${-motor_h/2-tube_off} 0 0" rpy="0 0 0" />
       <parent link="link1" />
       <child link="link2" />
-      <axis xyz="1 0 0" />
+      <axis xyz="-1 0 0" />
       <limit lower="${joint_limits['joint2']['min_position']}" upper="${joint_limits['joint2']['max_position']}"
       velocity="${joint_limits['joint2']['max_velocity']}" effort="100" />
@@ -108,9 +108,9 @@
     <xacro:property name="arm1_l" value="0.368" />
     <xacro:property name="arm1_m" value="${1650*(arm_r**2*pi-arm_ri**2*pi)*arm1_l}" />
-    <xacro:property name="arm2_l" value="0.307" />
+    <xacro:property name="arm2_l" value="0.28" />
     <xacro:property name="arm2_m" value="${1650*(arm_r**2*pi-arm_ri**2*pi)*arm2_l}" />
     <link name="link2">
       <visual>
-        <origin xyz="${arm_r} 0 ${-arm1_l/2}" rpy="0 0 0" />
+        <origin xyz="${-arm_r} 0 ${-arm1_l/2}" rpy="0 0 0" />
         <geometry>
           <cylinder length="${arm1_l}" radius="${arm_r}" />
@@ -119,5 +119,5 @@
       </visual>
       <collision>
-        <origin xyz="${arm_r} 0 ${-arm1_l/2}" rpy="0 0 0" />
+        <origin xyz="${-arm_r} 0 ${-arm1_l/2}" rpy="0 0 0" />
         <geometry>
           <cylinder length="${arm1_l}" radius="${arm_r}" />
@@ -125,5 +125,5 @@
       </collision>
       <inertial>
-        <origin xyz="${arm_r} 0 ${-arm1_l/2}" rpy="0 0 0" />
+        <origin xyz="${-arm_r} 0 ${-arm1_l/2}" rpy="0 0 0" />
         <mass value="${arm1_m}" />
         <xacro:cylinder_inertia m="${arm1_m}" r="${arm_r}" h="${arm1_l}" />
@@ -131,5 +131,5 @@
     </link>
     <joint name="joint2_motor" type="fixed">
-      <origin xyz="${-motor_h/2-0.0058} 0 ${-arm1_l}" rpy="0 0 0" />
+      <origin xyz="${motor_h/2+0.0058} 0 ${-arm1_l}" rpy="0 0 0" />
       <parent link="link2" />
       <child link="link2_motor" />
@@ -156,5 +156,5 @@
     </link>
     <joint name="joint3" type="revolute">
-      <origin xyz="${-motor_h/2-tube_off} 0 0" rpy="${pi} 0 0" />
+      <origin xyz="${motor_h/2+tube_off} 0 0" rpy="${pi} 0 0" />
       <parent link="link2_motor" />
       <child link="link3" />
@@ -165,5 +165,5 @@
     <link name="link3">
       <visual>
-        <origin xyz="${-arm_r} 0 ${-arm2_l/2}" rpy="0 0 0" />
+        <origin xyz="${arm_r} 0 ${-arm2_l/2}" rpy="0 0 0" />
         <geometry>
           <cylinder length="${arm2_l}" radius="${arm_r}" />
@@ -172,5 +172,5 @@
       </visual>
       <collision>
-        <origin xyz="${-arm_r} 0 ${-arm2_l/2}" rpy="0 0 0" />
+        <origin xyz="${arm_r} 0 ${-arm2_l/2}" rpy="0 0 0" />
         <geometry>
           <cylinder length="${arm2_l}" radius="${arm_r}" />
@@ -178,5 +178,5 @@
       </collision>
       <inertial>
-        <origin xyz="${-arm_r} 0 ${-arm2_l/2}" rpy="0 0 0" />
+        <origin xyz="${arm_r} 0 ${-arm2_l/2}" rpy="0 0 0" />
         <mass value="${arm2_m}" />
         <xacro:cylinder_inertia m="${arm2_m}" r="${arm_r}" h="${arm2_l}" />
@@ -184,5 +184,5 @@
     </link>
     <joint name="joint3_end" type="fixed">
-      <origin xyz="${-arm_r} 0 ${-arm2_l}" rpy="0 0 0" />
+      <origin xyz="${arm_r} 0 ${-arm2_l}" rpy="0 0 0" />
       <parent link="link3" />
       <child link="eef_link" />

Commit message: feat: update urdf

File: ofa_description/urdf/ofa_robot_description.urdf.xacro (robot description, xacro)
@@ -2,7 +2,41 @@
 <robot xmlns:xacro="http://www.ros.org/wiki/xacro">
   <xacro:macro name="weed_robot" params="parent">
+    <!-- Axis dimensions (box) -->
+    <xacro:property name="axis_l" value="1.216" />
+    <xacro:property name="axis_w" value="0.06" />
+    <xacro:property name="axis_h" value="0.072" />
+    <xacro:property name="axis_m" value="6" />
+    <!-- Distance between carriage hard stop and end of axis -->
+    <xacro:property name="carriage_off" value="${axis_l-0.116-1}" />
+    <!-- Distance between axis carriage and center of first motor -->
     <xacro:property name="attachment_off" value="${0.06+0.002}" />
+    <!-- Distance between ground and carriage -->
+    <xacro:property name="height" value="${0.65-axis_h}" />
+    <!-- Distance between motor and tube -->
     <xacro:property name="tube_off" value="${0.01}" />
-    <xacro:property name="height" value="${0.5+attachment_off}" />
+    <!-- Motor dimensions (cylinder) -->
+    <xacro:property name="motor_r" value="${0.089/2}" />
+    <xacro:property name="motor_h" value="0.05025" />
+    <xacro:property name="motor_m" value="0.521" />
+    <!-- Offset between center of motor and center of carriage in x-direction -->
+    <xacro:property name="motor_off" value="${0.0026}" />
+    <!-- Camera enclosure dimensions (box) -->
+    <xacro:property name="camera_w" value="0.12" />
+    <xacro:property name="camera_h" value="0.08" />
+    <xacro:property name="camera_l" value="0.048" />
+    <xacro:property name="camera_m" value="0.335" />
+    <!-- Offset between camera enclosure and motor center -->
+    <xacro:property name="camera_off" value="${motor_h/2+0.04355}" />
+    <!-- Tube dimensions (cylinders) -->
+    <xacro:property name="arm_r" value="${0.045/2}" />
+    <xacro:property name="arm_ri" value="${0.041/2}" />
+    <xacro:property name="arm1_l" value="0.368" />
+    <xacro:property name="arm1_m" value="${1650*(arm_r**2*pi-arm_ri**2*pi)*arm1_l}" />
+    <xacro:property name="arm2_l" value="0.28" />
+    <xacro:property name="arm2_m" value="${1650*(arm_r**2*pi-arm_ri**2*pi)*arm2_l}" />
+    <!-- End effector dimensions (cylinder) -->
+    <xacro:property name="end_r" value="0.005" />
+    <xacro:property name="end_l" value="0.02" />
+    <xacro:property name="end_m" value="1" />
     <joint name="base_joint" type="fixed">
       <origin xyz="0 0 ${height}" rpy="0 0 0" />
@@ -10,31 +44,26 @@
       <child link="base_link" />
     </joint>
-    <xacro:property name="base_l" value="1.216" />
-    <xacro:property name="base_w" value="0.06" />
-    <xacro:property name="base_h" value="0.072" />
-    <xacro:property name="base_m" value="6" />
     <link name="base_link">
       <visual>
-        <origin xyz="0 0 ${base_h/2}" rpy="0 0 0" />
-        <geometry>
-          <box size="${base_l} ${base_w} ${base_h}" />
+        <origin xyz="0 0 ${axis_h/2}" rpy="0 0 0" />
+        <geometry>
+          <box size="${axis_l} ${axis_w} ${axis_h}" />
         </geometry>
         <material name="blue"/>
       </visual>
       <collision>
-        <origin xyz="0 0 ${base_h/2}" rpy="0 0 0" />
-        <geometry>
-          <box size="${base_l} ${base_w} ${base_h}" />
-        </geometry>
-      </collision>
-      <inertial>
-        <origin xyz="0 0 ${base_h/2}" rpy="0 0 0" />
-        <mass value="${base_m}" />
-        <xacro:box_inertia m="${base_m}" x="${base_l}" y="${base_w}" z="${base_h}" />
-      </inertial>
-    </link>
-    <xacro:property name="axis_length" value="1" />
+        <origin xyz="0 0 ${axis_h/2}" rpy="0 0 0" />
+        <geometry>
+          <box size="${axis_l} ${axis_w} ${axis_h}" />
+        </geometry>
+      </collision>
+      <inertial>
+        <origin xyz="0 0 ${axis_h/2}" rpy="0 0 0" />
+        <mass value="${axis_m}" />
+        <xacro:box_inertia m="${axis_m}" x="${axis_l}" y="${axis_w}" z="${axis_h}" />
+      </inertial>
+    </link>
     <joint name="joint1" type="prismatic">
-      <origin xyz="${base_l/2-0.116} 0 ${-attachment_off}" rpy="0 0 0" />
+      <origin xyz="${axis_l/2-carriage_off+motor_off} 0 ${-attachment_off}" rpy="0 0 0" />
       <parent link="base_link" />
       <child link="link1" />
@@ -43,7 +72,4 @@
       velocity="${joint_limits['joint1']['max_velocity']}" effort="100" />
     </joint>
-    <xacro:property name="motor_r" value="${0.089/2}" />
-    <xacro:property name="motor_h" value="0.05025" />
-    <xacro:property name="motor_m" value="0.521" />
     <link name="link1">
       <visual>
@@ -66,9 +92,4 @@
       </inertial>
     </link>
-    <xacro:property name="camera_w" value="0.12" />
-    <xacro:property name="camera_h" value="0.08" />
-    <xacro:property name="camera_l" value="0.048" />
-    <xacro:property name="camera_m" value="0.335" />
-    <xacro:property name="camera_off" value="${0.0885/2+0.004}" />
     <joint name="joint1_camera" type="fixed">
       <origin xyz="${camera_off} 0 ${attachment_off}" rpy="0 0 0" />
@@ -104,10 +125,4 @@
       velocity="${joint_limits['joint2']['max_velocity']}" effort="100" />
     </joint>
-    <xacro:property name="arm_r" value="${0.045/2}" />
-    <xacro:property name="arm_ri" value="${0.041/2}" />
-    <xacro:property name="arm1_l" value="0.368" />
-    <xacro:property name="arm1_m" value="${1650*(arm_r**2*pi-arm_ri**2*pi)*arm1_l}" />
-    <xacro:property name="arm2_l" value="0.28" />
-    <xacro:property name="arm2_m" value="${1650*(arm_r**2*pi-arm_ri**2*pi)*arm2_l}" />
     <link name="link2">
       <visual>
@@ -131,5 +146,5 @@
     </link>
     <joint name="joint2_motor" type="fixed">
-      <origin xyz="${motor_h/2+0.0058} 0 ${-arm1_l}" rpy="0 0 0" />
+      <origin xyz="${motor_h/2+tube_off} 0 ${-arm1_l}" rpy="0 0 0" />
       <parent link="link2" />
       <child link="link2_motor" />
@@ -188,7 +203,4 @@
       <child link="eef_link" />
     </joint>
-    <xacro:property name="end_r" value="0.005" />
-    <xacro:property name="end_l" value="0.02" />
-    <xacro:property name="end_m" value="1" />
     <link name="eef_link">
       <visual>

Commit message: feat: position list move

File: ofa_description/urdf/ofa_robot_description.urdf.xacro (robot description, xacro)
@@ -40,5 +40,5 @@
     <xacro:property name="end_m" value="1" />
     <joint name="base_joint" type="fixed">
-      <origin xyz="0 0 ${height}" rpy="0 0 ${pi}" />
+      <origin xyz="0 0 ${height}" rpy="0 0 0" />
       <parent link="${parent}" />
       <child link="base_link" />

Commit message: fix: x direction

File: ofa_description/urdf/ofa_robot_description.urdf.xacro (robot description, xacro)
@@ -65,8 +65,8 @@
     </link>
     <joint name="joint1" type="prismatic">
-      <origin xyz="${axis_l/2-carriage_off+motor_off} 0 ${-attachment_off}" rpy="0 0 0" />
+      <origin xyz="${-axis_l/2+carriage_off-motor_off} 0 ${-attachment_off}" rpy="0 0 0" />
       <parent link="base_link" />
       <child link="link1" />
-      <axis xyz="1 0 0" />
+      <axis xyz="-1 0 0" />
       <limit lower="${joint_limits['joint1']['min_position']}" upper="${joint_limits['joint1']['max_position']}"
       velocity="${joint_limits['joint1']['max_velocity']}" effort="100" />
@@ -93,5 +93,5 @@
     </link>
     <joint name="joint1_camera" type="fixed">
-      <origin xyz="${camera_off} 0 ${attachment_off}" rpy="0 0 0" />
+      <origin xyz="${-camera_off} 0 ${attachment_off}" rpy="0 0 0" />
       <parent link="link1" />
       <child link="link1_camera" />
@@ -99,18 +99,18 @@
     <link name="link1_camera">
       <visual>
-        <origin xyz="${camera_l/2} 0 ${-camera_h/2}" rpy="0 0 0" />
+        <origin xyz="${-camera_l/2} 0 ${-camera_h/2}" rpy="0 0 0" />
+        <geometry>
+          <box size="${-camera_l} ${camera_w} ${camera_h}" />
+        </geometry>
+        <material name="grey"/>
+      </visual>
+      <collision>
+        <origin xyz="${-camera_l/2} 0 ${-camera_h/2}" rpy="0 0 0" />
         <geometry>
           <box size="${camera_l} ${camera_w} ${camera_h}" />
         </geometry>
-        <material name="grey"/>
-      </visual>
-      <collision>
-        <origin xyz="${camera_l/2} 0 ${-camera_h/2}" rpy="0 0 0" />
-        <geometry>
-          <box size="${camera_l} ${camera_w} ${camera_h}" />
-        </geometry>
-      </collision>
-      <inertial>
-        <origin xyz="${camera_l/2} 0 ${-camera_h/2}" rpy="0 0 0" />
+      </collision>
+      <inertial>
+        <origin xyz="${-camera_l/2} 0 ${-camera_h/2}" rpy="0 0 0" />
         <mass value="${camera_m}" />
         <xacro:box_inertia m="${camera_m}" x="${camera_l}" y="${camera_w}" z="${camera_h}" />
@@ -118,5 +118,5 @@
     </link>
     <joint name="joint2" type="revolute">
-      <origin xyz="${-motor_h/2-tube_off} 0 0" rpy="0 0 0" />
+      <origin xyz="${motor_h/2+tube_off} 0 0" rpy="0 0 0" />
       <parent link="link1" />
       <child link="link2" />
@@ -127,5 +127,5 @@
     <link name="link2">
       <visual>
-        <origin xyz="${-arm_r} 0 ${-arm1_l/2}" rpy="0 0 0" />
+        <origin xyz="${arm_r} 0 ${-arm1_l/2}" rpy="0 0 0" />
         <geometry>
           <cylinder length="${arm1_l}" radius="${arm_r}" />
@@ -134,5 +134,5 @@
       </visual>
       <collision>
-        <origin xyz="${-arm_r} 0 ${-arm1_l/2}" rpy="0 0 0" />
+        <origin xyz="${arm_r} 0 ${-arm1_l/2}" rpy="0 0 0" />
         <geometry>
           <cylinder length="${arm1_l}" radius="${arm_r}" />
@@ -140,5 +140,5 @@
       </collision>
       <inertial>
-        <origin xyz="${-arm_r} 0 ${-arm1_l/2}" rpy="0 0 0" />
+        <origin xyz="${arm_r} 0 ${-arm1_l/2}" rpy="0 0 0" />
         <mass value="${arm1_m}" />
         <xacro:cylinder_inertia m="${arm1_m}" r="${arm_r}" h="${arm1_l}" />
@@ -146,5 +146,5 @@
     </link>
     <joint name="joint2_motor" type="fixed">
-      <origin xyz="${motor_h/2+tube_off} 0 ${-arm1_l}" rpy="0 0 0" />
+      <origin xyz="${-motor_h/2-tube_off} 0 ${-arm1_l}" rpy="0 0 0" />
       <parent link="link2" />
       <child link="link2_motor" />
@@ -171,5 +171,5 @@
     </link>
     <joint name="joint3" type="revolute">
-      <origin xyz="${motor_h/2+tube_off} 0 0" rpy="${pi} 0 0" />
+      <origin xyz="${-motor_h/2-tube_off} 0 0" rpy="${pi} 0 0" />
       <parent link="link2_motor" />
       <child link="link3" />
@@ -180,5 +180,5 @@
     <link name="link3">
       <visual>
-        <origin xyz="${arm_r} 0 ${-arm2_l/2}" rpy="0 0 0" />
+        <origin xyz="${-arm_r} 0 ${-arm2_l/2}" rpy="0 0 0" />
         <geometry>
           <cylinder length="${arm2_l}" radius="${arm_r}" />
@@ -187,5 +187,5 @@
       </visual>
       <collision>
-        <origin xyz="${arm_r} 0 ${-arm2_l/2}" rpy="0 0 0" />
+        <origin xyz="${-arm_r} 0 ${-arm2_l/2}" rpy="0 0 0" />
         <geometry>
           <cylinder length="${arm2_l}" radius="${arm_r}" />
@@ -193,5 +193,5 @@
       </collision>
       <inertial>
-        <origin xyz="${arm_r} 0 ${-arm2_l/2}" rpy="0 0 0" />
+        <origin xyz="${-arm_r} 0 ${-arm2_l/2}" rpy="0 0 0" />
         <mass value="${arm2_m}" />
         <xacro:cylinder_inertia m="${arm2_m}" r="${arm_r}" h="${arm2_l}" />
@@ -199,5 +199,5 @@
     </link>
     <joint name="joint3_end" type="fixed">
-      <origin xyz="${arm_r} 0 ${-arm2_l}" rpy="0 0 0" />
+      <origin xyz="${-arm_r} 0 ${-arm2_l}" rpy="0 0 0" />
       <parent link="link3" />
       <child link="eef_link" />

Commit message: chore: cleanup

File: ofa_description/urdf/ofa_robot_description.urdf.xacro (robot description, xacro)
@@ -121,5 +121,5 @@
       <parent link="link1" />
       <child link="link2" />
-      <axis xyz="-1 0 0" />
+      <axis xyz="1 0 0" />
       <limit lower="${joint_limits['joint2']['min_position']}" upper="${joint_limits['joint2']['max_position']}"
       velocity="${joint_limits['joint2']['max_velocity']}" effort="100" />
@@ -174,5 +174,5 @@
       <parent link="link2_motor" />
       <child link="link3" />
-      <axis xyz="1 0 0" />
+      <axis xyz="-1 0 0" />
       <limit lower="${joint_limits['joint3']['min_position']}" upper="${joint_limits['joint3']['max_position']}"
       velocity="${joint_limits['joint3']['max_velocity']}" effort="100" />

Commit message: feat: camera block

File: ofa_description/urdf/ofa_robot_description.urdf.xacro (robot description, xacro)
@@ -26,6 +26,11 @@
     <xacro:property name="camera_l" value="0.048" />
     <xacro:property name="camera_m" value="0.335" />
+    <xacro:property name="camera_block_w" value="0.01" />
+    <xacro:property name="camera_block_h" value="0.08" />
+    <xacro:property name="camera_block_l" value="0.048" />
+    <xacro:property name="camera_block_m" value="0.01" />
     <!-- Offset between camera enclosure and motor center -->
-    <xacro:property name="camera_off" value="${motor_h/2+0.04355}" />
+    <xacro:property name="camera_off_x" value="${motor_h/2+0.04355}" />
+    <xacro:property name="camera_off_y" value="${0.044}" />
     <!-- Tube dimensions (cylinders) -->
     <xacro:property name="arm_r" value="${0.045/2}" />
@@ -33,9 +38,9 @@
     <xacro:property name="arm1_l" value="0.368" />
     <xacro:property name="arm1_m" value="${1650*(arm_r**2*pi-arm_ri**2*pi)*arm1_l}" />
-    <xacro:property name="arm2_l" value="0.28" />
+    <xacro:property name="arm2_l" value="0.17" />
     <xacro:property name="arm2_m" value="${1650*(arm_r**2*pi-arm_ri**2*pi)*arm2_l}" />
     <!-- End effector dimensions (cylinder) -->
-    <xacro:property name="end_r" value="0.005" />
-    <xacro:property name="end_l" value="0.02" />
+    <xacro:property name="end_r" value="0.01" />
+    <xacro:property name="end_l" value="0.2" />
     <xacro:property name="end_m" value="1" />
     <joint name="base_joint" type="fixed">
@@ -93,5 +98,5 @@
     </link>
     <joint name="joint1_camera" type="fixed">
-      <origin xyz="${-camera_off} 0 ${attachment_off}" rpy="0 0 0" />
+      <origin xyz="${-camera_off_x} ${-camera_off_y} ${attachment_off}" rpy="0 0 0" />
       <parent link="link1" />
       <child link="link1_camera" />
@@ -101,5 +106,5 @@
         <origin xyz="${-camera_l/2} 0 ${-camera_h/2}" rpy="0 0 0" />
         <geometry>
-          <box size="${-camera_l} ${camera_w} ${camera_h}" />
+          <box size="${camera_l} ${camera_w} ${camera_h}" />
         </geometry>
         <material name="grey"/>
@@ -115,4 +120,29 @@
         <mass value="${camera_m}" />
         <xacro:box_inertia m="${camera_m}" x="${camera_l}" y="${camera_w}" z="${camera_h}" />
+      </inertial>
+    </link>
+    <joint name="joint1_camera_block" type="fixed">
+      <origin xyz="0 ${-camera_w/2} 0" rpy="0 0 0" />
+      <parent link="link1_camera" />
+      <child link="link1_camera_block" />
+    </joint>
+    <link name="link1_camera_block">
+      <visual>
+        <origin xyz="${camera_block_l/2} ${camera_block_w/2} ${-camera_block_h/2}" rpy="0 0 0" />
+        <geometry>
+          <box size="${camera_block_l} ${camera_block_w} ${camera_block_h}" />
+        </geometry>
+        <material name="grey"/>
+      </visual>
+      <collision>
+        <origin xyz="${camera_block_l/2} ${camera_block_w/2} ${-camera_block_h/2}" rpy="0 0 0" />
+        <geometry>
+          <box size="${camera_block_l} ${camera_block_w} ${camera_block_h}" />
+        </geometry>
+      </collision>
+      <inertial>
+        <origin xyz="${camera_block_l/2} ${camera_block_w/2} ${-camera_block_h/2}" rpy="0 0 0" />
+        <mass value="${camera_block_m}" />
+        <xacro:box_inertia m="${camera_block_m}" x="${camera_block_l}" y="${camera_block_w}" z="${camera_block_h}" />
       </inertial>
     </link>
