Commit message: feat: update urdf

File: ofa_description/urdf/ofa_robot.urdf (robot description, URDF)
Before this commit: robot ofa_robot, 8 links, 7 joints
Links:
- removed link link1_camera
- added link camera_color_frame
- added link camera_link; collision box size=0.04026 0.11526 0.06525; visual box size=0.04026 0.11526 0.06525
- added link camera_shield_link; collision box size=0.048 0.002 0.08; collision box size=0.048 0.002 0.08
- link base_link: mass 6 -> None
- link eef_link: mass 1 -> None; geometry 
- link link1: mass 0.521 -> None
- link link2: mass 0.11144799938609781 -> None; geometry collision cylinder length=0.368 radius=0.0225; visual cylinder length=0.368 radius=0.0225
- link link2_motor: mass 0.521 -> None
- link link3: mass 0.18946159895636627 -> None; geometry collision cylinder length=0.05 radius=0.003; collision cylinder length=0.15 radius=0.013
Joints:
- removed joint joint1_camera
- added joint camera_color_joint: type fixed, parent camera_link, child camera_color_frame, origin xyz=0 0.03 -0.05659361 rpy=3.141592653589793 0 1.5707963267948966
- added joint camera_joint: type fixed, parent camera_shield_link, child camera_link, origin xyz=0 -0.00045 -0.00615 rpy=0 0 0
- added joint camera_shield_joint: type fixed, parent link1, child camera_shield_link, origin xyz=-0.09267500000000001 -0.044 0.062 rpy=0 0 0
- joint base_joint: origin xyz=0 0 0.562 rpy=0 0 0 -> xyz=0 0 0.5780000000000001 rpy=0 0 0
- joint joint1: axis 1 0 0 -> -1 0 0; limit lower=0.0 upper=1.0 effort=100 velocity=10.0 -> lower=-0.95 upper=0.0 effort=100 velocity=1.0; origin xyz=-0.492 0 -0.062 rpy=0 0 0 -> xyz=-0.5106000000000002 0 -0.062 rpy=0 0 0
- joint joint2: limit lower=-2.1 upper=2.1 effort=100 velocity=20.0 -> lower=-2.1 upper=2.1 effort=100 velocity=10.0; origin xyz=0.035125 0 0 rpy=0 0 0 -> xyz=0.057625 0 0 rpy=0 0 0
- joint joint2_motor: origin xyz=-0.030925 0 -0.25 rpy=0 0 0 -> xyz=-0.057625 0 -0.368 rpy=0 0 0
- joint joint3: axis 1 0 0 -> -1 0 0; limit lower=-2.1 upper=2.1 effort=100 velocity=20.0 -> lower=-2.1 upper=2.1 effort=100 velocity=10.0; origin xyz=-0.035125 0 0 rpy=0 0 0 -> xyz=-0.057625 0 0 rpy=3.141592653589793 0 0
- joint joint3_end: origin xyz=-0.0225 0 -0.425 rpy=0 0 0 -> xyz=0 0 -0.37 rpy=0 0 0

File: ofa_description/urdf/ofa_robot.urdf.xacro (robot description, xacro)
@@ -8,5 +8,4 @@
    <xacro:include filename="ofa_robot_description.urdf.xacro" />
   <!-- Import materials and inertia macros -->
-  <xacro:include filename="inertia.urdf.xacro" />
   <xacro:include filename="materials.urdf.xacro" />
   <!-- Import ros2_control description -->

File: ofa_description/urdf/ofa_robot_description.urdf.xacro (robot description, xacro)
@@ -6,5 +6,4 @@
     <xacro:property name="axis_w" value="0.06" />
     <xacro:property name="axis_h" value="0.072" />
-    <xacro:property name="axis_m" value="6" />
     <!-- Distance between carriage hard stop and end of axis -->
     <xacro:property name="carriage_off" value="${axis_l-0.116-1}" />
@@ -15,33 +14,35 @@
     <!-- Distance between motor and tube -->
     <xacro:property name="tube_off" value="${0.01}" />
-    <!-- Motor dimensions (cylinder) -->
+    <!-- Motor dimensions -->
     <xacro:property name="motor_r" value="${0.089/2}" />
     <xacro:property name="motor_h" value="0.05025" />
-    <xacro:property name="motor_m" value="0.521" />
     <!-- Offset between center of motor and center of carriage in x-direction -->
     <xacro:property name="motor_off" value="${0.0026}" />
-    <!-- Camera enclosure dimensions (box) -->
-    <xacro:property name="camera_w" value="0.12" />
-    <xacro:property name="camera_h" value="0.08" />
-    <xacro:property name="camera_l" value="0.048" />
-    <xacro:property name="camera_m" value="0.335" />
-    <xacro:property name="camera_block_w" value="0.01" />
-    <xacro:property name="camera_block_h" value="0.08" />
-    <xacro:property name="camera_block_l" value="0.048" />
-    <xacro:property name="camera_block_m" value="0.01" />
+    <!-- Camera enclosure dimensions -->
+    <xacro:property name="camera_shield_w" value="0.12" />
+    <xacro:property name="camera_shield_h" value="0.08" />
+    <xacro:property name="camera_shield_l" value="0.048" />
+    <xacro:property name="camera_shield_wall" value="0.002" />
     <!-- Offset between camera enclosure and motor center -->
-    <xacro:property name="camera_off_x" value="${motor_h/2+0.04355}" />
-    <xacro:property name="camera_off_y" value="${0.044}" />
-    <!-- Tube dimensions (cylinders) -->
+    <xacro:property name="camera_shield_off_x" value="${motor_h/2+0.04355}" />
+    <xacro:property name="camera_shield_off_y" value="${0.044}" />
+    <!-- Camera dimensions -->
+    <xacro:property name="camera_w" value="0.11526" />
+    <xacro:property name="camera_h" value="0.06525" />
+    <xacro:property name="camera_l" value="0.04026" />
+    <xacro:property name="camera_off_y" value="0.00045" />
+    <xacro:property name="camera_off_z" value="0.00615" />
+    <!-- Offset between camera and optical center of rgb camera -->
+    <xacro:property name="color_off_y" value="0.03" />
+    <xacro:property name="color_off_z" value="0.05659361" />
+    <!-- Tube dimensions -->
     <xacro:property name="arm_r" value="${0.045/2}" />
-    <xacro:property name="arm_ri" value="${0.041/2}" />
     <xacro:property name="arm1_l" value="0.368" />
-    <xacro:property name="arm1_m" value="${1650*(arm_r**2*pi-arm_ri**2*pi)*arm1_l}" />
     <xacro:property name="arm2_l" value="0.17" />
-    <xacro:property name="arm2_m" value="${1650*(arm_r**2*pi-arm_ri**2*pi)*arm2_l}" />
-    <!-- End effector dimensions (cylinder) -->
-    <xacro:property name="end_r" value="0.01" />
-    <xacro:property name="end_l" value="0.2" />
-    <xacro:property name="end_m" value="1" />
+    <!-- End effector dimensions -->
+    <xacro:property name="end_base_r" value="0.013" />
+    <xacro:property name="end_base_l" value="0.15" />
+    <xacro:property name="end_tip_r" value="0.003" />
+    <xacro:property name="end_tip_l" value="0.05" />
     <joint name="base_joint" type="fixed">
       <origin xyz="0 0 ${height}" rpy="0 0 0" />
@@ -63,9 +64,4 @@
         </geometry>
       </collision>
-      <inertial>
-        <origin xyz="0 0 ${axis_h/2}" rpy="0 0 0" />
-        <mass value="${axis_m}" />
-        <xacro:box_inertia m="${axis_m}" x="${axis_l}" y="${axis_w}" z="${axis_h}" />
-      </inertial>
     </link>
     <joint name="joint1" type="prismatic">
@@ -91,18 +87,48 @@
         </geometry>
       </collision>
-      <inertial>
-        <origin xyz="0 0 0" rpy="0 ${pi/2} 0" />
-        <mass value="${motor_m}" />
-        <xacro:cylinder_inertia m="${motor_m}" r="${motor_r}" h="${motor_h}" />
-      </inertial>
-    </link>
-    <joint name="joint1_camera" type="fixed">
-      <origin xyz="${-camera_off_x} ${-camera_off_y} ${attachment_off}" rpy="0 0 0" />
+    </link>
+    <joint name="camera_shield_joint" type="fixed">
+      <origin xyz="${-camera_shield_off_x-camera_shield_l/2} ${-camera_shield_off_y} ${attachment_off}" rpy="0 0 0" />
       <parent link="link1" />
-      <child link="link1_camera" />
-    </joint>
-    <link name="link1_camera">
-      <visual>
-        <origin xyz="${-camera_l/2} 0 ${-camera_h/2}" rpy="0 0 0" />
+      <child link="camera_shield_link" />
+    </joint>
+    <link name="camera_shield_link">
+      <visual>
+        <origin xyz="0 ${-camera_shield_w/2+camera_shield_wall/2} ${-camera_shield_h/2}" rpy="0 0 0" />
+        <geometry>
+          <box size="${camera_shield_l} ${camera_shield_wall} ${camera_shield_h}" />
+        </geometry>
+        <material name="grey"/>
+      </visual>
+      <visual>
+        <origin xyz="0 ${camera_shield_w/2-camera_shield_wall/2} ${-camera_shield_h/2}" rpy="0 0 0" />
+        <geometry>
+          <box size="${camera_shield_l} ${camera_shield_wall} ${camera_shield_h}" />
+        </geometry>
+        <material name="grey"/>
+      </visual>
+      <collision>
+        <origin xyz="0 ${-camera_shield_w/2+camera_shield_wall/2} ${-camera_shield_h/2}" rpy="0 0 0" />
+        <geometry>
+          <box size="${camera_shield_l} ${camera_shield_wall} ${camera_shield_h}" />
+        </geometry>
+        <material name="grey"/>
+      </collision>
+      <collision>
+        <origin xyz="0 ${camera_shield_w/2-camera_shield_wall/2} ${-camera_shield_h/2}" rpy="0 0 0" />
+        <geometry>
+          <box size="${camera_shield_l} ${camera_shield_wall} ${camera_shield_h}" />
+        </geometry>
+        <material name="grey"/>
+      </collision>
+    </link>
+    <joint name="camera_joint" type="fixed">
+      <origin xyz="0 ${-camera_off_y} ${-camera_off_z}" rpy="0 0 0" />
+      <parent link="camera_shield_link" />
+      <child link="camera_link" />
+    </joint>
+    <link name="camera_link">
+      <visual>
+        <origin xyz="0 0 ${-camera_h/2}" rpy="0 0 0" />
         <geometry>
           <box size="${camera_l} ${camera_w} ${camera_h}" />
@@ -111,42 +137,19 @@
       </visual>
       <collision>
-        <origin xyz="${-camera_l/2} 0 ${-camera_h/2}" rpy="0 0 0" />
+        <origin xyz="0 0 ${-camera_h/2}" rpy="0 0 0" />
         <geometry>
           <box size="${camera_l} ${camera_w} ${camera_h}" />
         </geometry>
-      </collision>
-      <inertial>
-        <origin xyz="${-camera_l/2} 0 ${-camera_h/2}" rpy="0 0 0" />
-        <mass value="${camera_m}" />
-        <xacro:box_inertia m="${camera_m}" x="${camera_l}" y="${camera_w}" z="${camera_h}" />
-      </inertial>
-    </link>
-    <joint name="joint1_camera_block" type="fixed">
-      <origin xyz="0 ${-camera_w/2} 0" rpy="0 0 0" />
-      <parent link="link1_camera" />
-      <child link="link1_camera_block" />
-    </joint>
-    <link name="link1_camera_block">
-      <visual>
-        <origin xyz="${camera_block_l/2} ${camera_block_w/2} ${-camera_block_h/2}" rpy="0 0 0" />
-        <geometry>
-          <box size="${camera_block_l} ${camera_block_w} ${camera_block_h}" />
-        </geometry>
-        <material name="grey"/>
-      </visual>
-      <collision>
-        <origin xyz="${camera_block_l/2} ${camera_block_w/2} ${-camera_block_h/2}" rpy="0 0 0" />
-        <geometry>
-          <box size="${camera_block_l} ${camera_block_w} ${camera_block_h}" />
-        </geometry>
-      </collision>
-      <inertial>
-        <origin xyz="${camera_block_l/2} ${camera_block_w/2} ${-camera_block_h/2}" rpy="0 0 0" />
-        <mass value="${camera_block_m}" />
-        <xacro:box_inertia m="${camera_block_m}" x="${camera_block_l}" y="${camera_block_w}" z="${camera_block_h}" />
-      </inertial>
-    </link>
+        <material name="grey"/>
+      </collision>
+    </link>
+    <joint name="camera_color_joint" type="fixed">
+      <origin xyz="0 ${color_off_y} ${-color_off_z}" rpy="${pi} 0 ${pi/2}" />
+      <parent link="camera_link" />
+      <child link="camera_color_frame" />
+    </joint>
+    <link name="camera_color_frame" />
     <joint name="joint2" type="revolute">
-      <origin xyz="${motor_h/2+tube_off} 0 0" rpy="0 0 0" />
+      <origin xyz="${motor_h/2+tube_off+arm_r} 0 0" rpy="0 0 0" />
       <parent link="link1" />
       <child link="link2" />
@@ -157,5 +160,5 @@
     <link name="link2">
       <visual>
-        <origin xyz="${arm_r} 0 ${-arm1_l/2}" rpy="0 0 0" />
+        <origin xyz="0 0 ${-arm1_l/2}" rpy="0 0 0" />
         <geometry>
           <cylinder length="${arm1_l}" radius="${arm_r}" />
@@ -164,17 +167,12 @@
       </visual>
       <collision>
-        <origin xyz="${arm_r} 0 ${-arm1_l/2}" rpy="0 0 0" />
+        <origin xyz="0 0 ${-arm1_l/2}" rpy="0 0 0" />
         <geometry>
           <cylinder length="${arm1_l}" radius="${arm_r}" />
         </geometry>
       </collision>
-      <inertial>
-        <origin xyz="${arm_r} 0 ${-arm1_l/2}" rpy="0 0 0" />
-        <mass value="${arm1_m}" />
-        <xacro:cylinder_inertia m="${arm1_m}" r="${arm_r}" h="${arm1_l}" />
-      </inertial>
     </link>
     <joint name="joint2_motor" type="fixed">
-      <origin xyz="${-motor_h/2-tube_off} 0 ${-arm1_l}" rpy="0 0 0" />
+      <origin xyz="${-motor_h/2-tube_off-arm_r} 0 ${-arm1_l}" rpy="0 0 0" />
       <parent link="link2" />
       <child link="link2_motor" />
@@ -194,12 +192,7 @@
         </geometry>
       </collision>
-      <inertial>
-        <origin xyz="0 0 0" rpy="0 ${pi/2} 0" />
-        <mass value="${motor_m}" />
-        <xacro:cylinder_inertia m="${motor_m}" r="${motor_r}" h="${motor_h}" />
-      </inertial>
     </link>
     <joint name="joint3" type="revolute">
-      <origin xyz="${-motor_h/2-tube_off} 0 0" rpy="${pi} 0 0" />
+      <origin xyz="${-motor_h/2-tube_off-arm_r} 0 0" rpy="${pi} 0 0" />
       <parent link="link2_motor" />
       <child link="link3" />
@@ -210,5 +203,5 @@
     <link name="link3">
       <visual>
-        <origin xyz="${-arm_r} 0 ${-arm2_l/2}" rpy="0 0 0" />
+        <origin xyz="0 0 ${-arm2_l/2}" rpy="0 0 0" />
         <geometry>
           <cylinder length="${arm2_l}" radius="${arm_r}" />
@@ -216,85 +209,45 @@
         <material name="orange"/>
       </visual>
-      <collision>
-        <origin xyz="${-arm_r} 0 ${-arm2_l/2}" rpy="0 0 0" />
+      <visual>
+        <origin xyz="0 0 ${-arm2_l-end_base_l/2}" rpy="0 0 0" />
+        <geometry>
+          <cylinder length="${end_base_l}" radius="${end_base_r}" />
+        </geometry>
+        <material name="orange"/>
+      </visual>
+      <visual>
+        <origin xyz="0 0 ${-arm2_l-end_base_l-end_tip_l/2}" rpy="0 0 0" />
+        <geometry>
+          <cylinder length="${end_tip_l}" radius="${end_tip_r}" />
+        </geometry>
+        <material name="orange"/>
+      </visual>
+      <collision>
+        <origin xyz="0 0 ${-arm2_l/2}" rpy="0 0 0" />
         <geometry>
           <cylinder length="${arm2_l}" radius="${arm_r}" />
         </geometry>
       </collision>
-      <inertial>
-        <origin xyz="${-arm_r} 0 ${-arm2_l/2}" rpy="0 0 0" />
-        <mass value="${arm2_m}" />
-        <xacro:cylinder_inertia m="${arm2_m}" r="${arm_r}" h="${arm2_l}" />
-      </inertial>
+      <collision>
+        <origin xyz="0 0 ${-arm2_l-end_base_l/2}" rpy="0 0 0" />
+        <geometry>
+          <cylinder length="${end_base_l}" radius="${end_base_r}" />
+        </geometry>
+        <material name="orange"/>
+      </collision>
+      <collision>
+        <origin xyz="0 0 ${-arm2_l-end_base_l-end_tip_l/2}" rpy="0 0 0" />
+        <geometry>
+          <cylinder length="${end_tip_l}" radius="${end_tip_r}" />
+        </geometry>
+        <material name="orange"/>
+      </collision>
     </link>
     <joint name="joint3_end" type="fixed">
-      <origin xyz="${-arm_r} 0 ${-arm2_l}" rpy="0 0 0" />
+      <origin xyz="0 0 ${-arm2_l-end_base_l-end_tip_l}" rpy="0 0 0" />
       <parent link="link3" />
       <child link="eef_link" />
     </joint>
-    <link name="eef_link">
-      <visual>
-        <origin xyz="0 0 ${-end_l/2}" rpy="0 0 0" />
-        <geometry>
-          <cylinder length="${end_l}" radius="${end_r}" />
-        </geometry>
-        <material name="black"/>
-      </visual>
-      <collision>
-        <origin xyz="0 0 ${-end_l/2}" rpy="0 0 0" />
-        <geometry>
-          <cylinder length="${end_l}" radius="${end_r}" />
-        </geometry>
-      </collision>
-      <inertial>
-        <origin xyz="0 0 ${-end_l/2}" rpy="0 0 0" />
-        <mass value="${end_m}" />
-        <xacro:cylinder_inertia m="${end_m}" r="${end_r}" h="${end_l}" />
-      </inertial>
-    </link>
+    <link name="eef_link" />
 	</xacro:macro>
-	<!-- <xacro:property name="top_l" value="0.2" />
-	<xacro:property name="top_w" value="0.2" />
-	<xacro:property name="wheel_r" value="0.2" />
-	<xacro:property name="wheel_l" value="0.1" />
-	<xacro:property name="wheel_m" value="5" />
-	<xacro:property name="top_h" value="${height-2*wheel_r}" />
-	<xacro:macro name="wheel" params="prefix x y">
-		<joint name="_wheel_joint" type="fixed">
-			<parent link="base_link" />
-			<child link="_wheel_link" />
-			<origin xyz="${x} ${y} 0" rpy="0 0 0" />
-		</joint>
-		<link name="_wheel_link">
-			<visual>
-				<origin xyz="0 0 ${-top_h/2}" rpy="0 0 0"/>
-				<geometry>
-					<box size="${top_l} ${top_w} ${top_h}" />
-				</geometry>
-				<material name="blue"/>
-			</visual>
-			<visual>
-				<origin xyz="0 0 ${-top_h-wheel_r}" rpy="${pi/2} 0 0"/>
-				<geometry>
-					<cylinder radius="${wheel_r}" length="${wheel_l}" />
-				</geometry>
-				<material name="blue"/>
-			</visual>
-			<collision>
-				<origin xyz="0 0 ${-top_h/2-wheel_r}" rpy="0 0 0"/>
-				<geometry>
-					<box size="${top_l} ${2*wheel_r} ${top_h+2*wheel_r}" />
-				</geometry>
-			</collision>
-			<inertial>
-				<origin xyz="0 0 ${-top_h/2-wheel_r}" rpy="0 0 0"/>
-				<mass value="${wheel_m}" />
-				<xacro:box_inertia m="${wheel_m}" x="${top_w}" y="${2*wheel_r}" z="${top_h+2*wheel_r}" />
-			</inertial>
-		</link>
-	</xacro:macro>
-	<xacro:wheel prefix="fl" x="${base_l/2-top_w/2}" y="${base_w/2-top_l/2}" />
-	<xacro:wheel prefix="bl" x="${-base_l/2+top_w/2}" y="${base_w/2-top_l/2}" />
-	<xacro:wheel prefix="fr" x="${base_l/2-top_w/2}" y="${-base_w/2+top_l/2}" />
-	<xacro:wheel prefix="br" x="${-base_l/2+top_w/2}" y="${-base_w/2+top_l/2}" /> -->
 </robot>

Commit message: feat: collision boxes

File: ofa_description/urdf/ofa_robot.urdf (robot description, URDF)
Before this commit: robot ofa_robot, 10 links, 9 joints
Links:
- link base_link: geometry collision box size=1.216 0.06 0.072; collision box size=1.3 0.01 0.68
Joints:
- joint base_joint: origin xyz=0 0 0.5780000000000001 rpy=0 0 0 -> xyz=0 0 0.68 rpy=0 0 0
- joint joint1: origin xyz=-0.5106000000000002 0 -0.062 rpy=0 0 0 -> xyz=-0.5106000000000002 0 -0.134 rpy=0 0 0

File: ofa_description/urdf/ofa_robot_description.urdf.xacro (robot description, xacro)
@@ -2,14 +2,27 @@
 <robot xmlns:xacro="http://www.ros.org/wiki/xacro">
   <xacro:macro name="weed_robot" params="parent">
-    <!-- Axis dimensions (box) -->
+    <!-- Axis dimensions -->
     <xacro:property name="axis_l" value="1.216" />
     <xacro:property name="axis_w" value="0.06" />
     <xacro:property name="axis_h" value="0.072" />
+    <!-- Collision boxes -->
+    <xacro:property name="frame_l" value="1.3" />
+    <xacro:property name="frame_w" value="0.9" />
+    <xacro:property name="frame_h" value="0.03" />
+    <xacro:property name="box_w" value="0.01" />
+    <!-- Side (Wheels) -->
+    <xacro:property name="frame_l" value="1.3" />
+    <xacro:property name="frame_w" value="0.8" />
+    <xacro:property name="frame_h" value="0.03" />
+    <!-- Frame dimensions -->
+    <xacro:property name="frame_l" value="1.3" />
+    <xacro:property name="frame_w" value="0.8" />
+    <xacro:property name="frame_h" value="0.03" />
     <!-- Distance between carriage hard stop and end of axis -->
     <xacro:property name="carriage_off" value="${axis_l-0.116-1}" />
     <!-- Distance between axis carriage and center of first motor -->
     <xacro:property name="attachment_off" value="${0.06+0.002}" />
-    <!-- Distance between ground and carriage -->
-    <xacro:property name="height" value="${0.65-axis_h}" />
+    <!-- Distance between ground and top of axis -->
+    <xacro:property name="height" value="${0.68}" />
     <!-- Distance between motor and tube -->
     <xacro:property name="tube_off" value="${0.01}" />
@@ -52,5 +65,5 @@
     <link name="base_link">
       <visual>
-        <origin xyz="0 0 ${axis_h/2}" rpy="0 0 0" />
+        <origin xyz="0 0 ${-axis_h/2}" rpy="0 0 0" />
         <geometry>
           <box size="${axis_l} ${axis_w} ${axis_h}" />
@@ -59,12 +72,39 @@
       </visual>
       <collision>
-        <origin xyz="0 0 ${axis_h/2}" rpy="0 0 0" />
+        <origin xyz="0 0 ${-axis_h/2}" rpy="0 0 0" />
         <geometry>
           <box size="${axis_l} ${axis_w} ${axis_h}" />
         </geometry>
       </collision>
+      <!-- Top (Frame) -->
+      <collision>
+        <origin xyz="0 0 ${-frame_h/2}" rpy="0 0 0" />
+        <geometry>
+          <box size="${frame_l} ${frame_w} ${frame_h}" />
+        </geometry>
+      </collision>
+      <!-- Side (Wheels) -->
+      <collision>
+        <origin xyz="0 ${-frame_w/2-box_w/2} ${-height/2}" rpy="0 0 0" />
+        <geometry>
+          <box size="${frame_l} ${box_w} ${height}" />
+        </geometry>
+      </collision>
+      <collision>
+        <origin xyz="0 ${frame_w/2+box_w/2} ${-height/2}" rpy="0 0 0" />
+        <geometry>
+          <box size="${frame_l} ${box_w} ${height}" />
+        </geometry>
+      </collision>
+      <!-- Bottom (Ground) -->
+      <collision>
+        <origin xyz="0 0 ${-height-box_w/2}" rpy="0 0 0" />
+        <geometry>
+          <box size="${frame_l} ${frame_w} ${box_w}" />
+        </geometry>
+      </collision>
     </link>
     <joint name="joint1" type="prismatic">
-      <origin xyz="${-axis_l/2+carriage_off-motor_off} 0 ${-attachment_off}" rpy="0 0 0" />
+      <origin xyz="${-axis_l/2+carriage_off-motor_off} 0 ${-axis_h-attachment_off}" rpy="0 0 0" />
       <parent link="base_link" />
       <child link="link1" />
@@ -113,5 +153,4 @@
           <box size="${camera_shield_l} ${camera_shield_wall} ${camera_shield_h}" />
         </geometry>
-        <material name="grey"/>
       </collision>
       <collision>
@@ -120,5 +159,4 @@
           <box size="${camera_shield_l} ${camera_shield_wall} ${camera_shield_h}" />
         </geometry>
-        <material name="grey"/>
       </collision>
     </link>
@@ -141,5 +179,4 @@
           <box size="${camera_l} ${camera_w} ${camera_h}" />
         </geometry>
-        <material name="grey"/>
       </collision>
     </link>
@@ -234,5 +271,4 @@
           <cylinder length="${end_base_l}" radius="${end_base_r}" />
         </geometry>
-        <material name="orange"/>
       </collision>
       <collision>
@@ -241,5 +277,4 @@
           <cylinder length="${end_tip_l}" radius="${end_tip_r}" />
         </geometry>
-        <material name="orange"/>
       </collision>
     </link>

Commit message: feat: update urdf

File: ofa_description/urdf/ofa_robot.urdf (robot description, URDF)
Before this commit: robot ofa_robot, 10 links, 9 joints
Links:
- link base_link: geometry collision box size=1.216 0.06 0.072; collision box size=1.3 0.01 0.75
- link link2: geometry collision cylinder length=0.362 radius=0.0225; visual cylinder length=0.362 radius=0.0225
- link link3: geometry collision cylinder length=0.034 radius=0.003; collision cylinder length=0.16 radius=0.013
Joints:
- joint base_joint: origin xyz=0 0 0.68 rpy=0 0 0 -> xyz=0 0 0.75 rpy=0 0 0
- joint joint2_motor: origin xyz=-0.057625 0 -0.368 rpy=0 0 0 -> xyz=-0.057625 0 -0.362 rpy=0 0 0
- joint joint3_end: origin xyz=0 0 -0.37 rpy=0 0 0 -> xyz=0 0 -0.355 rpy=0 0 0
