Commit message: docs: update readmes

File: ofa_moveit_config/urdf/ofa_robot_description.urdf.xacro (robot description, xacro)
@@ -12,8 +12,4 @@
   <xacro:property name="frame_h" value="0.03" />
   <xacro:property name="box_w" value="0.01" />
-  <!-- Side (Wheels) -->
-  <xacro:property name="frame_l" value="1.3" />
-  <xacro:property name="frame_w" value="0.8" />
-  <xacro:property name="frame_h" value="0.03" />
   <!-- Frame dimensions -->
   <xacro:property name="frame_l" value="1.3" />

Commit message: chore: update params

File: ofa_moveit_config/urdf/ofa_robot_description.urdf.xacro (robot description, xacro)
@@ -50,5 +50,5 @@
   <xacro:property name="arm_r" value="${0.045/2}" />
   <xacro:property name="arm1_l" value="${0.451-2*motor_r}" />
-  <xacro:property name="arm2_l" value="0.161" />
+  <xacro:property name="arm2_l" value="${0.1165+motor_r}" />
   <!-- End effector dimensions -->
   <xacro:property name="end_base_r" value="0.013" />

Commit message: feat: workspace limits

File: ofa_moveit_config/urdf/ofa_robot_description.urdf.xacro (robot description, xacro)
@@ -14,5 +14,5 @@
   <!-- Frame dimensions -->
   <xacro:property name="frame_l" value="1.3" />
-  <xacro:property name="frame_w" value="0.8" />
+  <xacro:property name="frame_w" value="1.0" />
   <xacro:property name="frame_h" value="0.03" />
   <!-- Distance between carriage hard stop and end of axis -->
